File: hardware/KiCad/airspeed.kicad_sch (KiCad schematic)
At the start: 4 parts, among them U1 4525DO-DS5AI001DP

Commit message: Update KiCad schematics and PCB footprints
Parts:
- C1: footprint Capacitor_SMD:C_0603_1608Metric_Pad1.08x0.95mm_HandSolder -> Capacitor_SMD:C_0201_0603Metric_Pad0.64x0.40mm_HandSolder
Changed lines of the file:
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@@
 			)
 		)
-		(property "Footprint" "Capacitor_SMD:C_0603_1608Metric_Pad1.08x0.95mm_HandSolder"
+		(property "Footprint" "Capacitor_SMD:C_0201_0603Metric_Pad0.64x0.40mm_HandSolder"
 			(at 112.7252 66.04 0)
 			(effects
