File: hardware/KiCad/lidar.kicad_sch (KiCad schematic)
At the start: 6 parts, among them J2 Conn_01x08, U3 TPS22919DCKT

Commit message: Update KiCad schematics and PCB footprints
Parts:
- C2: footprint Capacitor_SMD:C_0603_1608Metric_Pad1.08x0.95mm_HandSolder -> Capacitor_SMD:C_0201_0603Metric_Pad0.64x0.40mm_HandSolder
Connections:
- net LIDAR_RX: now also J2.2 (Pin_2); no longer J2.1 (Pin_1)
- net LIDAR_TX: now also J2.1 (Pin_1); no longer J2.2 (Pin_2)
Changed lines of the file:
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@@
 	(global_label "LIDAR_RX"
 		(shape output)
-		(at 115.57 76.2 180)
+		(at 115.57 78.74 180)
 		(fields_autoplaced yes)
 		(effects
@@
 		)
 		(property "Intersheetrefs" "${INTERSHEET_REFS}"
-			(at 108.5534 76.2 0)
+			(at 108.5534 78.74 0)
 			(effects
 				(font
@@
 	(global_label "LIDAR_TX"
 		(shape input)
-		(at 115.57 78.74 180)
+		(at 115.57 76.2 180)
 		(fields_autoplaced yes)
 		(effects
@@
 		)
 		(property "Intersheetrefs" "${INTERSHEET_REFS}"
-			(at 108.7348 78.74 0)
+			(at 108.7348 76.2 0)
 			(effects
 				(font
@@
 			)
 		)
-		(property "Footprint" "Capacitor_SMD:C_0603_1608Metric_Pad1.08x0.95mm_HandSolder"
+		(property "Footprint" "Capacitor_SMD:C_0201_0603Metric_Pad0.64x0.40mm_HandSolder"
 			(at 101.2952 100.33 0)
 			(effects
