File: hardware/KiCad/mcu_imu.kicad_sch (KiCad schematic)
At the start: 15 parts, among them SW1 RESET, SW2 SW_BOOT, SW3 USER_BUTTON, U2 ESP32-S3-WROOM-1U-N8R8, U4 BMI088

Commit message: Update KiCad schematics and PCB footprints
Parts:
- added J7: UART_PROG, Connector_PinHeader_2.54mm:PinHeader_1x04_P2.54mm_Vertical, symbol Connector_Generic:Conn_01x04
- added R15, R16: 10 K, Resistor_SMD:R_0603_1608Metric_Pad0.98x0.95mm_HandSolder, symbol Device:R
- C4, C5: value 100 nF -> 100nF; footprint Capacitor_SMD:C_0603_1608Metric_Pad1.08x0.95mm_HandSolder -> Capacitor_SMD:C_0201_0603Metric_Pad0.64x0.40mm_HandSolder
- C6: value 1 uF -> 1uF
- C7: value 0.1uF -> 100nF; footprint Capacitor_SMD:C_0603_1608Metric_Pad1.08x0.95mm_HandSolder -> Capacitor_SMD:C_0201_0603Metric_Pad0.64x0.40mm_HandSolder
- R2: value 1K -> 470
Connections:
- net +3.3V: now also R15.1, R16.1
- net GND: now also J7.2 (Pin_2)
- net at SW2.2, U2.27 (IO0): now also R15.2
- net at SW3.2, U2.22 (IO14): now also R16.2
- net RXDO: now reaches U2.36 (RXD0)
- net RXDO: now also J7.4 (Pin_4)
- net TXDO: now reaches U2.37 (TXD0)
- net TXDO: now also J7.3 (Pin_3)
- new net +5V: J7.1 (Pin_1)
- no-connect marks 19 -> 17
Other:
- moved on the sheet: SW2, SW3
