File: hardware/KiCad/power.kicad_sch (KiCad schematic)
At the start: 22 parts, among them J1 USB_C_Receptacle_USB2.0_16P, J3 Conn_01x02, U5 MCP73831-2-OT, U6 LM27313XMF

Commit message: Save remaining power schematic changes
Parts:
- renumbered PS1 to U7
Changed lines of the file:
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@@
 		(dnp no)
 		(fields_autoplaced yes)
-		(property "Reference" "PS1"
+		(property "Reference" "U7"
 			(at 59.69 144.78 0)
 			(effects
@@
 			(project ""
 				(path "/f5466e30-9697-4c42-96e2-a6468d9cb39f/5efe4031-5539-44e6-8b44-0d1eeefb4a3a"
-					(reference "PS1")
+					(reference "U7")
 					(unit 1)
 				)

Commit message: Update KiCad schematics and PCB footprints
Parts:
- added C17: 1uF, Capacitor_SMD:C_0603_1608Metric_Pad1.08x0.95mm_HandSolder, symbol Device:C
- added C18: 10uF, Capacitor_SMD:C_0805_2012Metric_Pad1.18x1.45mm_HandSolder, symbol Device:C
- added TP1: 3V3_TEST, TestPoint:TestPoint_Pad_D1.5mm, symbol Connector:TestPoint
- added TP2: 5V_TEST, TestPoint:TestPoint_Pad_D1.5mm, symbol Connector:TestPoint
- added TP3: VBAT_TEST, TestPoint:TestPoint_Pad_D1.5mm, symbol Connector:TestPoint
- added TP4: GND_TEST, TestPoint:TestPoint_Pad_D1.5mm, symbol Connector:TestPoint
- C12: value 2.2uF -> 1uF
- C15: value 22uF -> 10uF
Connections:
- net +3.3V: now also C18.2, TP1.1
- net +5V: now also TP2.1
- net GND: now also C17.2, C18.1, TP4.1
- net VBAT: now also C17.1, TP3.1
Other:
- moved on the sheet: C10, C11, C14, C15, R8
